File: kicad/pmt-control.kicad_pcb (KiCad board)
At the start: 2 copper layers, 91.4 x 66 mm, 30 parts, among them J1 Barrel_Jack, J2 AVR-ISP-6, SW1 Rotary_Encoder_Switch, U1 ATmega328-PU, U2 MB85RS256B, U3 MAX6951, Y1 8MHz

Commit message: schematic
Parts:
- removed C2: 22u, Capacitor_SMD:C_1206_3216Metric_Pad1.33x1.80mm_HandSolder
- removed C5, C6: 20p, Capacitor_SMD:C_1206_3216Metric_Pad1.33x1.80mm_HandSolder
- removed C7: 100n, Capacitor_SMD:C_1206_3216Metric_Pad1.33x1.80mm_HandSolder
- removed D6: CDBHM260L-HF, footprints:SOIC245P670X290-4N
- removed J2: AVR-ISP-6, Connector_PinHeader_2.54mm:PinHeader_2x03_P2.54mm_Vertical
- removed PS1: VXO7803-500-M, footprints:CONV_VXO7805-500-M
- removed Y1: 8MHz, Crystal:Crystal_HC49-U_Vertical
- added Q1: 2N7000, Package_TO_SOT_SMD:SOT-23_Handsoldering, F.Cu at (168.2, 94.5)
- added Q2: 2N7000, Package_TO_SOT_SMD:SOT-23_Handsoldering, F.Cu at (176.6, 87.7)
- added SW2: TTL, footprints:SW_PTS526_SM08_SMTR2_LFS, F.Cu at (41.9, 101.6)
- added SW3: RST, footprints:SW_PTS526_SM08_SMTR2_LFS, F.Cu at (48.7, 90.2)
- added U4: LM285Z-2.5, Package_TO_SOT_THT:TO-92_Inline, F.Cu at (175.3, 82.9)
- C1: value 10u -> 100nF
- J1: value Barrel_Jack -> OUT; footprint Connector_BarrelJack:BarrelJack_Horizontal -> Connector_Molex:Molex_KK-254_AE-6410-04A_1x04_P2.54mm_Vertical
- R1: value 100 -> R_US
- R3: value 1M -> R_US
- R4: value 4.7k -> R_US
- U1: value ATmega328-PU -> Pico; footprint Package_DIP:DIP-28_W7.62mm -> footprints:RPi_Pico_SMD_TH
- U2: value MB85RS256B -> AD5761BRUZ-AD5761BRUZ; footprint Package_SO:SOP-8_5.28x5.23mm_P1.27mm -> Package_SO:TSSOP-16_4.4x5mm_P0.65mm
- moved C1 121.3 mm to (182.9, 81.3)
- moved D1 120.6 mm to (182.9, 84.7)
- moved R1 104.2 mm to (174.0, 98.4), turned to 0 degrees
- moved R3 81.5 mm to (182.8, 88.0), turned to 0 degrees
- moved J1 66.3 mm to (139.7, 85.1)
- moved R4 51.8 mm to (180.4, 91.6), turned to 0 degrees
- moved U2 39.8 mm to (127.0, 92.7)
- moved R2 38.0 mm to (116.5, 90.8), turned to 0 degrees
- moved U1 35.8 mm to (81.3, 81.9), turned to 0 degrees
- moved C4 30.0 mm to (118.9, 84.1), turned to 0 degrees
- moved U3 25.2 mm to (111.7, 85.8)
- moved C3 21.6 mm to (110.5, 90.8), turned to 0 degrees
Connections:
- C1 pad 1: +VDC -> +5V
- D1 pad 1: GND -> Net-(D1-Pad1)
- J1 pad 1: Net-(D6-Pad3) -> GND
- J1 pad 2: Net-(D6-Pad4) -> Net-(J1-Pad2)
- J1 pad 3: (no net) -> Net-(J1-Pad3)
- R1 pad 1: +3V3 -> +5V
- R1 pad 2: Net-(D1-Pad2) -> Net-(R1-Pad2)
- R3 pad 1: Net-(C5-Pad2) -> +5V
- R3 pad 2: Net-(C6-Pad2) -> Net-(D1-Pad2)
- R4 pad 1: Net-(J2-Pad5) -> +5V
- R4 pad 2: +3V3 -> Net-(J1-Pad2)
- U1 pad 1: Net-(J2-Pad5) -> Net-(U1-Pad1)
- U1 pad 10: Net-(C6-Pad2) -> Net-(U1-Pad10)
- U1 pad 11: (no net) -> Net-(U1-Pad11)
- U1 pad 12: (no net) -> Net-(U1-Pad12)
- U1 pad 13: (no net) -> GND
- U1 pad 14: (no net) -> Net-(U1-Pad14)
- U1 pad 16: /7seg/~CS~ -> Net-(U1-Pad16)
- U1 pad 17: SCK -> Net-(U1-Pad17)
- U1 pad 18: MISO -> GND
- U1 pad 19: MOSI -> Net-(SW1-PadA)
- U1 pad 2: Net-(SW1-PadA) -> Net-(U1-Pad2)
- U1 pad 20: (no net) -> Net-(SW1-PadB)
- U1 pad 21: (no net) -> MISO
- U1 pad 22: GND -> Net-(U1-Pad22)
- U1 pad 23: (no net) -> GND
- U1 pad 24: (no net) -> SCK
- U1 pad 25: (no net) -> MOSI
- U1 pad 26: (no net) -> /7seg/~CS~
- U1 pad 27: (no net) -> Net-(Q1-Pad1)
- U1 pad 28: (no net) -> GND
- U1 pad 3: Net-(SW1-PadB) -> GND
- U1 pad 4: (no net) -> Net-(U1-Pad4)
- U1 pad 5: (no net) -> Net-(U1-Pad5)
- U1 pad 6: (no net) -> Net-(U1-Pad6)
- U1 pad 7: +3V3 -> Net-(U1-Pad7)
- U1 pad 9: Net-(C5-Pad2) -> Net-(SW2-Pad2)
- U2 pad 1: Net-(U1-Pad15) -> Net-(U1-Pad5)
- U2 pad 2: MISO -> Net-(U1-Pad6)
- U2 pad 3: (no net) -> Net-(U1-Pad7)
- U2 pad 4: GND -> Net-(R1-Pad2)
- U2 pad 5: MOSI -> GND
- U2 pad 6: SCK -> GND
- U2 pad 7: +3V3 -> Net-(J1-Pad3)
- U2 pad 8: +3V3 -> +5V
Routing:
- net +3V3: track 139.9 -> 0.00 mm, vias 1 -> 0
- net SCK: track 106.3 -> 0.00 mm, vias 2 -> 0
- net MOSI: track 100.7 -> 0.00 mm, vias 1 -> 0
- net MISO: track 60.6 -> 0.00 mm, vias 2 -> 0
- net /7seg/~CS~: track 46.4 -> 0.00 mm, vias 1 -> 0
- net Net-(C6-Pad2): track 30.3 -> 0.00 mm
- net Net-(C5-Pad2): track 27.0 -> 0.00 mm
- net Net-(SW1-PadA): track 21.4 -> 0.00 mm
- net /7seg/SEG1: track 72.6 -> 51.4 mm, vias 5 -> 4
- net Net-(SW1-PadB): track 20.2 -> 0.00 mm
- net /7seg/SEG3: track 61.9 -> 42.2 mm, vias 5 -> 4
- net Net-(J2-Pad5): track 19.6 -> 0.00 mm
- net /7seg/SEG0: track 64.5 -> 45.2 mm, vias 5 -> 4
- net /7seg/SEG6: track 59.8 -> 41.6 mm, vias 6 -> 4
- net /7seg/SEG8: track 65.8 -> 48.2 mm, vias 5 -> 4
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Other:
- board text added: "BLAISE THOMPSON UW MADISON WRIGHT GROUP"
- board text removed: "3.3V ONLY"
- board text removed: "9 to 30V"
- board text removed: "BLAISE THOMPSON UW MADISON INSTRUMENT SHOP"
- board text removed: "POWER"

Commit message: from leo
Parts:
- moved R1 84.8 mm to (98.0, 60.7)
- moved D1 53.7 mm to (131.1, 98.6)
- moved C1 51.1 mm to (131.8, 80.8)
- moved R4 49.2 mm to (131.8, 84.1)
- moved Q1 46.1 mm to (122.2, 93.7)
- moved Q2 45.9 mm to (131.1, 93.7)
- moved R3 45.8 mm to (138.2, 98.6), turned to 180 degrees
- moved U4 44.4 mm to (133.3, 68.6), turned to 270 degrees
- moved SW2 33.3 mm to (63.5, 76.2)
- moved C4 17.8 mm to (103.1, 92.2)
- moved SW3 15.2 mm to (63.5, 86.4)
- moved U2 10.8 mm to (123.4, 82.5)
- moved C3 10.1 mm to (111.5, 80.8)
- moved U3 7.97 mm to (104.1, 83.3), turned to 90 degrees
- moved R2 6.99 mm to (111.5, 85.9)
Routing:
- net Net-(U1-Pad4): track 0.00 -> 122.4 mm, vias 0 -> 1
- net +5V: track 0.00 -> 120.9 mm, vias 0 -> 2
- net Net-(U1-Pad7): track 0.00 -> 93.3 mm
- net GND: track 0.00 -> 92.7 mm, vias 0 -> 2
- net Net-(U1-Pad6): track 0.00 -> 92.5 mm
- net Net-(U1-Pad5): track 0.00 -> 92.4 mm
- net Net-(R1-Pad2): track 0.00 -> 72.4 mm, vias 0 -> 1
- net Net-(SW3-Pad1): track 0.00 -> 64.7 mm, vias 0 -> 1
- net +3V3: track 0.00 -> 64.0 mm, vias 0 -> 3
- net Net-(SW1-PadA): track 0.00 -> 63.3 mm
- net SCK: track 0.00 -> 56.0 mm, vias 0 -> 2
- net Net-(SW1-PadB): track 0.00 -> 55.1 mm
- net MOSI: track 0.00 -> 50.3 mm, vias 0 -> 2
- net MISO: track 0.00 -> 45.2 mm, vias 0 -> 2
- net Net-(Q1-Pad1): track 0.00 -> 41.3 mm, vias 0 -> 1
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